File: shield2.sch (KiCad schematic (older format))
At the start: 35 parts, among them J10 Conn_01x02, J100 GROVE, J11 Conn_01x15, J12 Conn_01x15, J70 GROVE, J80 GROVE, J90 GROVE, U10 MCP73831-2

Commit message: rev1
Parts:
- added Q10: Si2323, Package_TO_SOT_SMD:SOT-23, symbol _transistors:Si2323
Connections:
- net +BATT: now also Q10.3 (D); no longer J11.15 (Pin_15)
- net at D10.1 (K), R10.1: now also Q10.1 (G)
- new net VIN: J11.15 (Pin_15), Q10.2 (S)
Other:
- moved on the sheet: R12, R13
Changed lines of the file:
@@
 	0    -1   1    0
 $EndComp
-Text Notes 5650 5600 0    50   ~ 0
+Text Notes 5200 4200 0    50   ~ 0
 10K -  100mA\n 5K -  200mA\n 2K -  500mA\n 1K - 1000mA
 $Comp
@@
 L power:+BATT #PWR0161
 U 1 1 5D6162D6
-P 6300 4450
-F 0 "#PWR0161" H 6300 4300 50  0001 C CNN
-F 1 "+BATT" H 6315 4623 50  0000 C CNN
-F 2 "" H 6300 4450 50  0001 C CNN
-F 3 "" H 6300 4450 50  0001 C CNN
-	1    6300 4450
+P 6600 4450
+F 0 "#PWR0161" H 6600 4300 50  0001 C CNN
+F 1 "+BATT" H 6615 4623 50  0000 C CNN
+F 2 "" H 6600 4450 50  0001 C CNN
+F 3 "" H 6600 4450 50  0001 C CNN
+	1    6600 4450
 	1    0    0    -1
 $EndComp
@@
 $EndComp
 Wire Wire Line
-	6300 4500 6750 4500
+	6300 4500 6600 4500
 Wire Wire Line
 	6700 4650 6700 4600
@@
 L power:+BATT #PWR0163
 U 1 1 5D61DD3B
-P 6700 5150
-F 0 "#PWR0163" H 6700 5000 50  0001 C CNN
-F 1 "+BATT" H 6715 5323 50  0000 C CNN
-F 2 "" H 6700 5150 50  0001 C CNN
-F 3 "" H 6700 5150 50  0001 C CNN
-	1    6700 5150
+P 3800 5700
+F 0 "#PWR0163" H 3800 5550 50  0001 C CNN
+F 1 "+BATT" H 3815 5873 50  0000 C CNN
+F 2 "" H 3800 5700 50  0001 C CNN
+F 3 "" H 3800 5700 50  0001 C CNN
+	1    3800 5700
 	1    0    0    -1
 $EndComp
@@
 L Device:R_Small R?
 U 1 1 5D61E0F8
-P 6700 5300
+P 3800 5850
 AR Path="/5D61E0F8" Ref="R?"  Part="1"
 AR Path="/5D5E5D45/5D61E0F8" Ref="R12"  Part="1"
-F 0 "R12" H 6500 5350 50  0000 L CNN
-F 1 "100K" H 6450 5250 50  0000 L CNN
-F 2 "Resistor_SMD:R_0402_1005Metric" H 6700 5300 50  0001 C CNN
-F 3 "~" H 6700 5300 50  0001 C CNN
-	1    6700 5300
+F 0 "R12" H 3600 5900 50  0000 L CNN
+F 1 "100K" H 3550 5800 50  0000 L CNN
+F 2 "Resistor_SMD:R_0402_1005Metric" H 3800 5850 50  0001 C CNN
+F 3 "~" H 3800 5850 50  0001 C CNN
+	1    3800 5850
 	-1   0    0    -1
 $EndComp
@@
 L Device:R_Small R?
 U 1 1 5D61E481
-P 6700 5600
+P 3800 6150
 AR Path="/5D61E481" Ref="R?"  Part="1"
 AR Path="/5D5E5D45/5D61E481" Ref="R13"  Part="1"
-F 0 "R13" H 6500 5650 50  0000 L CNN
-F 1 "100K" H 6450 5550 50  0000 L CNN
-F 2 "Resistor_SMD:R_0402_1005Metric" H 6700 5600 50  0001 C CNN
-F 3 "~" H 6700 5600 50  0001 C CNN
-	1    6700 5600
+F 0 "R13" H 3600 6200 50  0000 L CNN
+F 1 "100K" H 3550 6100 50  0000 L CNN
+F 2 "Resistor_SMD:R_0402_1005Metric" H 3800 6150 50  0001 C CNN
+F 3 "~" H 3800 6150 50  0001 C CNN
+	1    3800 6150
 	-1   0    0    -1
 $EndComp
@@
 L power:GND #PWR?
 U 1 1 5D61E65D
-P 6700 5750
+P 3800 6300
 AR Path="/5D61E65D" Ref="#PWR?"  Part="1"
 AR Path="/5D5E5D45/5D61E65D" Ref="#PWR0164"  Part="1"
-F 0 "#PWR0164" H 6700 5500 50  0001 C CNN
-F 1 "GND" H 6705 5577 50  0000 C CNN
-F 2 "" H 6700 5750 50  0001 C CNN
-F 3 "" H 6700 5750 50  0001 C CNN
-	1    6700 5750
-	1    0    0    -1
-$EndComp
-Wire Wire Line
-	6700 5750 6700 5700
-Wire Wire Line
-	6700 5500 6700 5450
-Wire Wire Line
-	6700 5200 6700 5150
-Wire Wire Line
-	6700 5450 7150 5450
-Connection ~ 6700 5450
-Wire Wire Line
-	6700 5450 6700 5400
-Text Label 7150 5450 2    50   ~ 0
+F 0 "#PWR0164" H 3800 6050 50  0001 C CNN
+F 1 "GND" H 3805 6127 50  0000 C CNN
+F 2 "" H 3800 6300 50  0001 C CNN
+F 3 "" H 3800 6300 50  0001 C CNN
+	1    3800 6300
+	1    0    0    -1
+$EndComp
+Wire Wire Line
+	3800 6300 3800 6250
+Wire Wire Line
+	3800 6050 3800 6000
+Wire Wire Line
+	3800 5750 3800 5700
+Wire Wire Line
+	3800 6000 4250 6000
+Connection ~ 3800 6000
+Wire Wire Line
+	3800 6000 3800 5950
+Text Label 4250 6000 2    50   ~ 0
 V_DIV
 Wire Wire Line
@@
 Text Label 3100 1750 0    50   ~ 0
 D6
-$Comp
-L power:+BATT #PWR0165
-U 1 1 5D697F2D
-P 2000 2700
-F 0 "#PWR0165" H 2000 2550 50  0001 C CNN
-F 1 "+BATT" H 2015 2873 50  0000 C CNN
-F 2 "" H 2000 2700 50  0001 C CNN
-F 3 "" H 2000 2700 50  0001 C CNN
-	1    2000 2700
-	1    0    0    -1
-$EndComp
-Wire Wire Line
-	1750 2550 1800 2550
-Wire Wire Line
-	1800 2550 1800 2750
-Wire Wire Line
-	1800 2750 2000 2750
-Wire Wire Line
-	2000 2750 2000 2700
 $Comp
 L Device:D_Zener_Small D71
@@
 Text Label 2050 2150 2    50   ~ 0
 V_DIV
-Wire Wire Line
-	6300 4450 6300 4500
+$Comp
+L _transistors:Si2323 Q10
+U 1 1 5D55385D
+P 6500 5300
+F 0 "Q10" H 6705 5346 50  0000 L CNN
+F 1 "Si2323" H 6705 5255 50  0000 L CNN
+F 2 "Package_TO_SOT_SMD:SOT-23" H 6700 5225 50  0001 L CIN
+F 3 "http://www.farnell.com/datasheets/2046026.pdf?_ga=2.233127902.1310620760.1565599800-307862962.1549974152&_gac=1.83736036.1565357378.Cj0KCQjws7TqBRDgARIsAAHLHP6Ff0ggAHsX5ovTw6Mr__z9rSr27-wh8EBEzq7YQDg2BU0HYsvy7sEaAvtgEALw_wcB" H 6500 5300 50  0001 L CNN
+	1    6500 5300
+	1    0    0    -1
+$EndComp
+Wire Wire Line
+	4850 4800 4850 5300
+Wire Wire Line
+	4850 5300 6300 5300
+Connection ~ 4850 4800
+Wire Wire Line
+	6600 4500 6600 5100
+Connection ~ 6600 4500
+Wire Wire Line
+	6600 4500 6750 4500
+Wire Wire Line
+	6600 4450 6600 4500
+Text GLabel 6750 5500 2    50   Input ~ 0
+VIN
+Wire Wire Line
+	6600 5500 6750 5500
+Text GLabel 1900 2550 2    50   Input ~ 0
+VIN
+Wire Wire Line
+	1750 2550 1900 2550
 $EndSCHEMATC
